Commit message: feat: 完善双足步态训练与多地形流程

File: squat_training/retargeting/models/lyt/lyt_14dof.urdf (robot description, URDF)
Before this commit: robot lyt_14dof, 15 links, 14 joints
Joints:
- joint ankle_angle_l: limit lower=-0.5 upper=0.7 effort=500 velocity=10 -> lower=-0.349066 upper=0.785398 effort=500 velocity=10
- joint ankle_angle_r: limit lower=-0.5 upper=0.7 effort=500 velocity=10 -> lower=-0.349066 upper=0.785398 effort=500 velocity=10
- joint hip_adduction_l: limit lower=-0.524 upper=0.2 effort=500 velocity=10 -> lower=-0.188496 upper=0.036652 effort=500 velocity=10
- joint hip_adduction_r: limit lower=-0.524 upper=0.2 effort=500 velocity=10 -> lower=-0.188496 upper=0.036652 effort=500 velocity=10
- joint hip_flexion_l: limit lower=-0.787 upper=0.787 effort=500 velocity=10 -> lower=-0.223402 upper=0.422369 effort=500 velocity=10
- joint hip_flexion_r: limit lower=-0.787 upper=0.787 effort=500 velocity=10 -> lower=-0.223402 upper=0.422369 effort=500 velocity=10
- joint hip_rotation_l: limit lower=-2.0944 upper=2.0944 effort=500 velocity=10 -> lower=-0.148353 upper=0.013963 effort=500 velocity=10
- joint hip_rotation_r: limit lower=-2.0944 upper=2.0944 effort=500 velocity=10 -> lower=-0.148353 upper=0.013963 effort=500 velocity=10
- joint knee_angle_l: limit lower=-2 upper=0 effort=1000 velocity=10 -> lower=-1.047198 upper=0.209440 effort=1000 velocity=10
- joint knee_angle_r: limit lower=-2 upper=0 effort=1000 velocity=10 -> lower=-1.047198 upper=0.209440 effort=1000 velocity=10
- joint subtalar_angle_l: limit lower=-1 upper=1 effort=300 velocity=10 -> lower=-0.261799 upper=0.349066 effort=300 velocity=10
- joint subtalar_angle_r: limit lower=-1 upper=1 effort=300 velocity=10 -> lower=-0.261799 upper=0.349066 effort=300 velocity=10
